File: BetetrDom.kicad_pcb (KiCad board)
At the start: 4 copper layers, 75 parts, among them IC1 SiC437BED-T1-GE3, J1 XT60PW-M, J2 Raspberry_Pi_2_3, J4 Barrel_Jack_Switch, Q1 PXP012-30QLJ, Q2 PXP012-30QLJ, U2 LTC4412xS6

Commit message: update 2 everything is fixed
Parts:
- R4, R5: footprint Resistor_SMD:R_2010_5025Metric_Pad1.40x2.65mm_HandSolder -> Resistor_SMD:R_0402_1005Metric
- R6: footprint Resistor_SMD:R_0603_1608Metric_Pad0.98x0.95mm_HandSolder -> Resistor_SMD:R_0402_1005Metric
- RV1, RV10, RV11, RV12, RV2, RV3, RV4, RV5, RV6, RV7, RV8, RV9: footprint iclr:SDR1307A101K -> Resistor_SMD:R_0805_2012Metric
- moved A2 145.8 mm to (99.0, 54.0)
- moved A1 91.2 mm to (99.0, 31.0)
- moved RV7 32.3 mm to (186.5, 112.5)
- moved L6 4.70 mm to (179.5, 24.5)
- moved L9 1.50 mm to (183.0, 51.0)
Connections:
- TP5 pad 1: unconnected-(TP5-Pad1) -> Net-(J2-ID_SC/GPIO1)
- TP6 pad 1: unconnected-(TP6-Pad1) -> Net-(J2-ID_SC/GPIO1)

Commit message: ideal diode update to be checked
Parts:
- added J3: XT60PW-M, iclr:AMASS_XT60PW-M, F.Cu at (39.0, 89.5)
- moved J1 188.2 mm to (39.0, 105.5), turned to 90 degrees
- moved A2 52.3 mm to (77.5, 6.34)
- moved A1 24.9 mm to (97.7, 6.11)
Connections:
- C5 pad 1: Net-(Q2-S_1) -> Net-(J3-+)
- Q2 pad 1: Net-(Q2-S_1) -> Net-(J3-+)

Commit message: update again
Parts:
- moved U2 171.1 mm to (57.1, 104.0)
Connections:
- C5 pad 1: Net-(J3-+) -> /+BATTV
- J3 pad 1: Net-(J3-+) -> /+BATTV
- Q2 pad 1: Net-(J3-+) -> /+BATTV
Changed lines of the file:
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@@
 	(net 79 "unconnected-(Q2-D_3-Pad7)")
 	(net 80 "Net-(Q2-G)")
-	(net 81 "Net-(J3-+)")
 	(footprint "TestPoint:TestPoint_Pad_1.5x1.5mm"
 		(layer "F.Cu")
@@
 	(footprint "Package_TO_SOT_SMD:TSOT-23-6"
 		(layer "F.Cu")
-		(at 223.525 64.35)
+		(at 57.1375 104.05)
 		(descr "TSOT, 6 Pin (https://www.jedec.org/sites/default/files/docs/MO-193D.pdf variant AA), generated with kicad-footprint-generator ipc_gullwing_generator.py")
 		(tags "TSOT TO_SOT_SMD")
@@
 			(size 0.4 0.6)
 			(layers "F.Cu" "F.Paste" "F.Mask")
-			(net 81 "Net-(J3-+)")
+			(net 4 "/+BATTV")
 			(pinfunction "S_1")
 			(pintype "passive")
@@
 			(layers "F.Cu" "F.Paste" "F.Mask")
 			(roundrect_rratio 0.25)
-			(net 81 "Net-(J3-+)")
+			(net 4 "/+BATTV")
 			(pintype "passive")
 		)
@@
 			(layers "*.Cu" "*.Mask")
 			(remove_unused_layers no)
-			(net 81 "Net-(J3-+)")
+			(net 4 "/+BATTV")
 			(pinfunction "+")
 			(pintype "passive")

Commit message: update
Parts:
- removed C5: 0.1uF, Capacitor_SMD:C_0402_1005Metric
- removed J3: XT60PW-M, iclr:AMASS_XT60PW-M
- added C23: 0.1uF, Capacitor_SMD:C_0402_1005Metric, F.Cu at (49.5, 77.0)
- J4: value Barrel_Jack_Switch -> XT60PW-M; footprint Connector_BarrelJack:BarrelJack_Wuerth_6941xx301002 -> iclr:AMASS_XT60PW-M
- moved R2 184.3 mm to (56.1, 86.0), turned to 90 degrees
- moved J4 171.4 mm to (39.0, 73.5), turned to 90 degrees
- moved Q2 168.9 mm to (57.7, 91.0), turned to -90 degrees
- moved Q1 162.6 mm to (57.7, 80.5), turned to -90 degrees
- moved C6 155.5 mm to (69.5, 88.0), turned to -90 degrees
- moved IC1 118.7 mm to (127.0, 129.8)
- moved U2 29.1 mm to (55.4, 75.0)
- moved J1 16.0 mm to (39.0, 89.5)
Connections:
- J4 pad 1: Net-(Q2-S_1) -> Net-(J4-+)
- J4 pad 2: GND -> Net-(J4--)
- Q1 pad 1: /+BATTV -> Net-(J4-+)
- U2 pad 1: /+BATTV -> Net-(J4-+)

Commit message: finished pcb layouts, ready for check p sure
Parts:
- added C5: 0.1uF, Capacitor_SMD:C_0402_1005Metric, F.Cu at (69.5, 132.6)
- added H1: MountingHole_Pad, MountingHole:MountingHole_3.2mm_M3_DIN965_Pad, F.Cu at (143.0, 139.0)
- added H2: MountingHole_Pad, MountingHole:MountingHole_3.2mm_M3_DIN965_Pad, F.Cu at (52.8, 139.4)
- added H3: MountingHole_Pad, MountingHole:MountingHole_3.2mm_M3_DIN965_Pad, F.Cu at (80.0, 53.0)
- added H4: MountingHole_Pad, MountingHole:MountingHole_3.2mm_M3_DIN965_Pad, F.Cu at (143.0, 53.0)
- C10, C12: footprint Capacitor_SMD:C_0603_1608Metric -> Capacitor_SMD:C_0402_1005Metric
- R1: footprint Resistor_SMD:R_0805_2012Metric -> Resistor_SMD:R_0402_1005Metric
- R3: footprint iclr:ERJHP6D1000V -> Resistor_SMD:R_1206_3216Metric
- moved RV5 154.1 mm to (131.4, 64.0)
- moved RV3 153.1 mm to (116.4, 64.0)
- moved C1 150.5 mm to (101.0, 123.3), turned to -90 degrees
- moved C2 147.4 mm to (103.0, 123.3), turned to -90 degrees
- moved RV11 147.4 mm to (98.5, 64.0)
- moved C7 146.4 mm to (107.0, 132.1), turned to -90 degrees
- moved RV9 146.2 mm to (83.6, 64.0)
- moved C4 144.2 mm to (111.6, 132.1), turned to -90 degrees
- moved C10 143.1 mm to (112.5, 122.8), turned to 90 degrees
- moved C12 142.8 mm to (112.5, 124.7), turned to 90 degrees
- moved C8 142.7 mm to (109.3, 132.1), turned to -90 degrees
- moved RV12 140.8 mm to (109.1, 64.2)
- moved RV10 139.9 mm to (94.3, 64.0)
- moved RV6 137.8 mm to (141.9, 64.0)
- moved C9 137.1 mm to (113.9, 132.1), turned to -90 degrees
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Connections:
- net /power/SW_6 renamed /power/SW
- net Net-(A1-1A) renamed /StepperA/1A
- net Net-(A1-2B) renamed /StepperA/2B
- net Net-(A2-1A) renamed /StepperB/1A
- net Net-(A2-2B) renamed /StepperB/2B
- A1 pad 4: Net-(A1-1B) -> /StepperA/1B
- A1 pad 6: Net-(A1-2A) -> /StepperA/2A
- A1 pad 8: /+BATTV -> VMAIN
- A2 pad 4: Net-(A2-1B) -> /StepperB/1B
- A2 pad 6: Net-(A2-2A) -> /StepperB/2A
- A2 pad 8: /+BATTV -> VMAIN
- C1 pad 1: VCC -> VMAIN
- C10 pad 2: A_GND -> GND
- C13 pad 2: /StepperB/MB1 -> /StepperB/MA2
- C15 pad 2: /StepperB/MA2 -> /StepperB/MB1
- C17 pad 2: /StepperA/MB1 -> /StepperA/MA2
- C19 pad 2: /StepperA/MA2 -> /StepperA/MB1
- C2 pad 1: VCC -> VMAIN
- C3 pad 1: A_GND -> GND
- C3 pad 2: VCC -> VMAIN
- C6 pad 1: VCC -> VMAIN
- D3 pad 1: /StepperA/MA2 -> /StepperA/MB1
- D4 pad 1: /StepperB/MA2 -> /StepperB/MB1
- D7 pad 1: /StepperA/MB1 -> /StepperA/MA2
- D8 pad 1: /StepperB/MB1 -> /StepperB/MA2
- IC1 pad 1: VCC -> VMAIN
- IC1 pad 16: A_GND -> GND
- IC1 pad 2: VCC -> VMAIN
- IC1 pad 22: unconnected-(IC1-VIN_1-Pad22) -> /power/VIN
- IC1 pad 25: A_GND -> GND
- IC1 pad 26: unconnected-(IC1-VIN_2-Pad26) -> /power/VIN
- J1 pad 1: /+BATTV -> /power/+BATTV
- J1 pad 2: GND -> Net-(J1--)
- L2 pad 1: Net-(A2-1B) -> /StepperB/2A
- L2 pad 2: /StepperB/MB1 -> /StepperB/MA2
- L4 pad 1: Net-(A2-2A) -> /StepperB/1B
- L4 pad 2: /StepperB/MA2 -> /StepperB/MB1
- L6 pad 1: Net-(A1-1B) -> /StepperA/2A
- L6 pad 2: /StepperA/MB1 -> /StepperA/MA2
- L8 pad 1: Net-(A1-2A) -> /StepperA/1B
- L8 pad 2: /StepperA/MA2 -> /StepperA/MB1
- Q1 pad 8: VCC -> VMAIN
- Q2 pad 1: /+BATTV -> /power/+BATTV
- Q2 pad 8: VCC -> VMAIN
- R1 pad 2: A_GND -> GND
- R2 pad 2: VCC -> VMAIN
- R5 pad 2: A_GND -> GND
- RV1 pad 1: /StepperB/MB1 -> /StepperB/MA2
- RV11 pad 2: /StepperA/MA2 -> /StepperA/MB1
- RV2 pad 1: /StepperB/MA2 -> /StepperB/MB1
- RV3 pad 2: /StepperB/MB1 -> /StepperB/MA2
- RV5 pad 2: /StepperB/MA2 -> /StepperB/MB1
- RV7 pad 1: /StepperA/MB1 -> /StepperA/MA2
- RV8 pad 1: /StepperA/MA2 -> /StepperA/MB1
- RV9 pad 2: /StepperA/MB1 -> /StepperA/MA2
- StepperConnector1 pad 2: /StepperA/MB2 -> /StepperA/MA1
- StepperConnector1 pad 3: /StepperA/MA1 -> /StepperA/MB1
- StepperConnector1 pad 4: /StepperA/MB1 -> /StepperA/MB2
- StepperConnector2 pad 2: /StepperB/MB2 -> /StepperB/MA1
- StepperConnector2 pad 3: /StepperB/MA1 -> /StepperB/MB1
- StepperConnector2 pad 4: /StepperB/MB1 -> /StepperB/MB2
- U2 pad 6: VCC -> VMAIN
Routing:
- net VMAIN: track 0.00 -> 62.0 mm, vias 0 -> 8
- net /Step1: track 0.00 -> 46.4 mm, vias 0 -> 2
- net GND: track 0.00 -> 42.2 mm, vias 0 -> 35
- net /Dir2: track 0.00 -> 31.5 mm, vias 0 -> 2
- net /StepperA/MB2: track 0.00 -> 28.2 mm, vias 0 -> 3
- net /StepperB/MB2: track 0.00 -> 28.0 mm, vias 0 -> 3
- net /Dir1: track 0.00 -> 27.8 mm
- net /StepperA/MA2: track 0.00 -> 25.6 mm, vias 0 -> 3
- net /StepperB/MA1: track 0.00 -> 24.6 mm, vias 0 -> 3
- net /StepperB/MA2: track 0.00 -> 24.1 mm, vias 0 -> 3
- net /StepperA/MB1: track 0.00 -> 23.9 mm, vias 0 -> 3
- net /StepperB/MB1: track 0.00 -> 23.6 mm, vias 0 -> 3
- net /StepperA/MA1: track 0.00 -> 23.5 mm, vias 0 -> 3
- net Net-(J4-+): track 0.00 -> 21.7 mm
- net /Step2: track 0.00 -> 18.1 mm
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- added copper zone on B.Cu, net (none)
- added copper zone on F.Cu, net (none)
- added copper zone on B.Cu, net +3V3
- added copper zone on F.Cu, net +3V3
- added copper zone on B.Cu, net /StepperA/1A
- added copper zone on F.Cu, net /StepperA/1A
- added copper zone on B.Cu, net /StepperA/1B
- added copper zone on F.Cu, net /StepperA/1B
- added copper zone on B.Cu, net /StepperA/2A
- added copper zone on F.Cu, net /StepperA/2A
- added copper zone on B.Cu, net /StepperA/2B
- added copper zone on F.Cu, net /StepperA/2B
- added copper zone on B.Cu, net /StepperA/MA1
- added copper zone on F.Cu, net /StepperA/MA1
- added copper zone on B.Cu, net /StepperA/MA2
- added copper zone on F.Cu, net /StepperA/MA2
- added copper zone on B.Cu, net /StepperA/MB1
- added copper zone on F.Cu, net /StepperA/MB1
- added copper zone on B.Cu, net /StepperA/MB2
- added copper zone on F.Cu, net /StepperA/MB2
- added copper zone on B.Cu, net /StepperB/1A
- added copper zone on F.Cu, net /StepperB/1A
- added copper zone on B.Cu, net /StepperB/1B
- added copper zone on F.Cu, net /StepperB/1B
- added copper zone on B.Cu, net /StepperB/2A
- added copper zone on F.Cu, net /StepperB/2A
- added copper zone on B.Cu, net /StepperB/2B
- added copper zone on F.Cu, net /StepperB/2B
- added copper zone on B.Cu, net /StepperB/MA1
- added copper zone on F.Cu, net /StepperB/MA1
- added copper zone on B.Cu, net /StepperB/MA2
- added copper zone on F.Cu, net /StepperB/MA2
- added copper zone on B.Cu, net /StepperB/MB1
- added copper zone on F.Cu, net /StepperB/MB1
- added copper zone on B.Cu, net /StepperB/MB2
- added copper zone on F.Cu, net /StepperB/MB2
- added copper zone on B.Cu, net /power/+V_BUCK
- added copper zone on F.Cu, net /power/+V_BUCK
- added copper zone on In2.Cu, net /power/+V_BUCK
- added copper zone on B.Cu, net /power/SW
- added copper zone on F.Cu, net /power/SW
- added copper zone on B.Cu, net /power/V_OUT
- added copper zone on F.Cu, net /power/V_OUT
- added copper zone on B.Cu, net GND
- added copper zone on F.Cu, net GND
- added copper zone on In1.Cu, net GND
- added copper zone on B.Cu, net VMAIN
- added copper zone on F.Cu, net VMAIN
Other:
- board outline added: 98 x 94.3 mm

Commit message: no message
Parts:
- moved C4 0.60 mm to (111.6, 132.7)
- moved C7 0.60 mm to (107.0, 132.7)
- moved C8 0.60 mm to (109.3, 132.7)
- moved C9 0.60 mm to (113.9, 132.7)
Routing:
- net /power/SW: vias 1 -> 0
Changed lines of the file:
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@@
 	(footprint "Capacitor_SMD:C_1206_3216Metric"
 		(layer "F.Cu")
-		(at 113.9 132.125 -90)
+		(at 113.9 132.725 -90)
 		(descr "Capacitor SMD 1206 (3216 Metric), square (rectangular) end terminal, IPC_7351 nominal, (Body size source: IPC-SM-782 page 76, https://www.pcb-3d.com/wordpress/wp-content/uploads/ipc-sm-782a_amendment_1_and_2.pdf), generated with kicad-footprint-generator")
 		(tags "capacitor")
@@
 	(footprint "Capacitor_SMD:C_1206_3216Metric"
 		(layer "F.Cu")
-		(at 107 132.125 -90)
+		(at 107 132.725 -90)
 		(descr "Capacitor SMD 1206 (3216 Metric), square (rectangular) end terminal, IPC_7351 nominal, (Body size source: IPC-SM-782 page 76, https://www.pcb-3d.com/wordpress/wp-content/uploads/ipc-sm-782a_amendment_1_and_2.pdf), generated with kicad-footprint-generator")
 		(tags "capacitor")
@@
 	(footprint "Capacitor_SMD:C_1206_3216Metric"
 		(layer "F.Cu")
-		(at 109.3 132.125 -90)
+		(at 109.3 132.725 -90)
 		(descr "Capacitor SMD 1206 (3216 Metric), square (rectangular) end terminal, IPC_7351 nominal, (Body size source: IPC-SM-782 page 76, https://www.pcb-3d.com/wordpress/wp-content/uploads/ipc-sm-782a_amendment_1_and_2.pdf), generated with kicad-footprint-generator")
 		(tags "capacitor")
@@
 	(footprint "Capacitor_SMD:C_1206_3216Metric"
 		(layer "F.Cu")
-		(at 111.6 132.125 -90)
+		(at 111.6 132.725 -90)
 		(descr "Capacitor SMD 1206 (3216 Metric), square (rectangular) end terminal, IPC_7351 nominal, (Body size source: IPC-SM-782 page 76, https://www.pcb-3d.com/wordpress/wp-content/uploads/ipc-sm-782a_amendment_1_and_2.pdf), generated with kicad-footprint-generator")
 		(tags "capacitor")
@@
 		(net 20)
 	)
-	(via
-		(at 106.825 125.925)
-		(size 0.6)
-		(drill 0.3)
-		(layers "F.Cu" "B.Cu")
-		(free yes)
-		(net 20)
-	)
 	(segment
 		(start 106.9 119.95)
@@
 		(polygon
 			(pts
-				(xy 86.77 118.09) (xy 85.27 81.734521) (xy 82.150684 81.871008) (xy 81.83 118.03) (xy 81 118) (xy 81 120.75)
-				(xy 84.5 120.75) (xy 84.5 128.5) (xy 90.1 128.55) (xy 95.75 128.5) (xy 95.75 123.25) (xy 101 123.3)
-				(xy 103 123.3) (xy 104.5 123.35) (xy 106.65 123.1) (xy 106.65 120.7) (xy 105 120.65) (xy 105.63 118.22)
+				(xy 88.75 118) (xy 85.5 107.5) (xy 85.27 81.734521) (xy 82.150684 81.871008) (xy 81.83 118.03) (xy 81 118)
+				(xy 81 120.75) (xy 84.5 120.75) (xy 84.5 128.5) (xy 90.1 128.55) (xy 95.75 128.5) (xy 95.75 123.25)
+				(xy 101 123.3) (xy 103 123.3) (xy 104.5 123.35) (xy 106.65 123.1) (xy 106.65 120.7) (xy 105 120.65)
+				(xy 105.63 118.22)
 			)
 		)
@@
 			(pts
 				(xy 113.5 118.5) (xy 113.525 119.625) (xy 111.2 119.625) (xy 111.2 115.8) (xy 123.575 116.125) (xy 124.725 125.85)
-				(xy 124.65 133.925) (xy 116.2 133.8) (xy 115.85 132.075) (xy 113.9 132.125) (xy 107 132.125) (xy 105.3 132.225)
+				(xy 124.65 133.925) (xy 116.2 133.8) (xy 115.85 132.075) (xy 113.9 132.375) (xy 107 132.375) (xy 105.3 132.225)
 				(xy 105.4 129.375) (xy 108.3 129.45) (xy 108.3 127.85) (xy 108.325 126.5) (xy 113.7 126.45) (xy 115.875 119.55)
 				(xy 115.85 117.225) (xy 113.5 117.25)
