File: BetetrDom.kicad_pcb (KiCad board)
At the start: 4 copper layers, 98 x 94.3 mm, 84 parts, among them IC1 SiC437BED-T1-GE3, J1 XT60PW-M, J2 Raspberry_Pi_2_3, J4 XT60PW-M, Q1 PXP012-30QLJ, Q2 PXP012-30QLJ, U2 LTC4412xS6

Commit message: update-i hate babs
Parts:
- removed H1: MountingHole_Pad, MountingHole:MountingHole_3.2mm_M3_DIN965_Pad
- added H4: MountingHole_Pad, MountingHole:MountingHole_3.2mm_M3_DIN965_Pad, F.Cu at (153.0, 140.0)
- added H4: MountingHole_Pad, MountingHole:MountingHole_3.2mm_M3_DIN965_Pad, F.Cu at (153.1, 82.0)
- added H4: MountingHole_Pad, MountingHole:MountingHole_3.2mm_M3_DIN965_Pad, F.Cu at (201.1, 82.0)
- L1: value 1.5uH -> 3.3uH; footprint Inductor_SMD:L_1008_2520Metric -> iclr:IND_SPM10065VT-3R3M-D
- moved RV7 43.9 mm to (85.2, 76.7)
- moved RV1 43.9 mm to (120.3, 76.6)
- moved RV8 43.6 mm to (102.6, 76.5)
- moved RV2 43.5 mm to (137.5, 76.5)
- moved D4 42.9 mm to (106.4, 71.2), turned to 135 degrees
- moved D5 42.8 mm to (116.6, 71.1), turned to 45 degrees
- moved D1 42.2 mm to (82.5, 70.5), turned to 45 degrees
- moved C19 42.2 mm to (95.5, 75.2)
- moved RV11 42.2 mm to (95.6, 73.5)
- moved D3 42.2 mm to (95.7, 70.4)
- moved RV3 42.1 mm to (114.4, 73.5), turned to -45 degrees
- moved D2 42.1 mm to (92.3, 70.4)
- moved C18 42.1 mm to (92.1, 75.2)
- moved D8 42.1 mm to (139.5, 70.3), turned to 135 degrees
- moved RV10 42.1 mm to (92.3, 73.5)
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Connections:
- C23 pad 1: /power/gnd_buff -> /power/V_BASE
- C5 pad 1: /gnd_buff -> /power/+BATTV
- J1 pad 2: /gnd_buff -> GND
- J4 pad 2: /power/gnd_buff -> GND
Routing:
- net /Dir1: track 26.8 -> 57.9 mm
- net /StepperA/MB2: track 19.7 -> 0.00 mm, vias 3 -> 0
- net /StepperB/MA1: track 16.8 -> 0.00 mm, vias 2 -> 0
- net /StepperA/MA1: track 16.8 -> 0.00 mm
- net /StepperA/MA2: track 16.5 -> 0.00 mm, vias 3 -> 0
- net /Step1: track 45.4 -> 61.9 mm, vias 2 -> 0
- net /StepperB/MA2: track 16.2 -> 0.00 mm, vias 1 -> 0
- net /StepperB/MB1: track 15.8 -> 0.00 mm, vias 1 -> 0
- net /StepperA/MB1: track 15.8 -> 0.08 mm, vias 3 -> 0
- net /StepperB/MB2: track 15.7 -> 0.00 mm, vias 2 -> 0
- net /Dir2: track 31.5 -> 17.4 mm, vias 2 -> 0
- net GND: track 34.4 -> 21.1 mm, vias 67 -> 62
- net /StepperA/2B: track 7.05 -> 0.00 mm
- net /power/gnd_buff: track 4.84 -> 0.00 mm
- net /power/V_OUT: track 3.51 -> 0.00 mm
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- added copper zone on In2.Cu, net +3V3
- added copper zone on F.Cu, net Net-(IC1-FB)
- removed copper zone on B.Cu, net +3V3
- removed copper zone on F.Cu, net +3V3
- removed copper zone on B.Cu, net /StepperA/1A
- removed copper zone on B.Cu, net /StepperA/1B
- removed copper zone on B.Cu, net /StepperA/2A
- removed copper zone on B.Cu, net /StepperA/2B
- removed copper zone on B.Cu, net /StepperB/1A
- removed copper zone on B.Cu, net /StepperB/1B
- removed copper zone on B.Cu, net /StepperB/2A
- removed copper zone on B.Cu, net /StepperB/2B
- removed copper zone on F.Cu, net /gnd_buff
- removed copper zone on In2.Cu, net /power/+V_BUCK
- removed copper zone on B.Cu, net /power/SW
- removed copper zone on B.Cu, net /power/V_OUT
- removed copper zone on F.Cu, net /power/gnd_buff
Other:
- board size 98 x 94.3 mm -> 155 x 83.5 mm

Commit message: babs (barbara) jeng
Parts:
- moved H4 0.10 mm to (201.0, 82.0)
Changed lines of the file:
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@@
 	(footprint "MountingHole:MountingHole_3.2mm_M3_DIN965_Pad"
 		(layer "F.Cu")
-		(at 201.1 82)
+		(at 201 82)
 		(descr "Mounting Hole 3.2mm, M3, DIN965")
 		(tags "mounting hole 3.2mm m3 din965")

Commit message: fuck it baseball hat
Parts:
- J2: moved to B.Cu
- moved H4 113.0 mm to (104.0, 140.0)
- moved J2 2.55 mm to (151.6, 86.9), turned to 180 degrees
- moved G*** 1.10 mm to (111.4, 96.0)
Routing:
- net /Step1: track 61.9 -> 110.2 mm
- net /Step2: track 20.9 -> 24.4 mm
- net /Dir2: track 17.4 -> 20.8 mm
- net /Dir1: track 57.9 -> 60.4 mm
Other:
- board size 155 x 83.5 mm -> 108 x 83.5 mm

Commit message: donedonedone
Parts:
- Q1, Q2: value PXP012-30QLJ -> SQS141ELNW-T1_GE3; footprint iclr:PXP01230QLJ -> iclr:SQS850ENT1_GE3
- moved G*** 52.0 mm to (89.3, 100.6)
- moved G*** 24.2 mm to (91.5, 140.0) (x2)
- moved G*** 24.2 mm to (61.3, 140.0) (x2)
- moved Q2 3.55 mm to (77.0, 123.8), turned to 180 degrees
- moved Q1 1.80 mm to (77.3, 115.0), turned to 180 degrees
Connections:
- H4 pad 1: (no net) -> GND (x3)
- IC1 pad 22: /power/VIN -> VMAIN
- IC1 pad 26: /power/VIN -> VMAIN
- Q1 pad 1: /power/V_BASE -> VMAIN
- Q1 pad 2: unconnected-(Q1-S_2-Pad2) -> VMAIN
- Q1 pad 3: unconnected-(Q1-S_3-Pad3) -> VMAIN
- Q1 pad 5: unconnected-(Q1-D_1-Pad5) -> /power/V_BASE
- Q1 pad 6: unconnected-(Q1-D_2-Pad6) -> /power/V_BASE
- Q1 pad 7: unconnected-(Q1-D_3-Pad7) -> /power/V_BASE
- Q1 pad 8: VMAIN -> /power/V_BASE
- Q1 pad 9: unconnected-(Q1-D_5-Pad9) -> /power/V_BASE
- Q2 pad 1: /power/+BATTV -> VMAIN
- Q2 pad 2: unconnected-(Q2-S_2-Pad2) -> VMAIN
- Q2 pad 3: unconnected-(Q2-S_3-Pad3) -> VMAIN
- Q2 pad 5: unconnected-(Q2-D_1-Pad5) -> /power/+BATTV
- Q2 pad 6: unconnected-(Q2-D_2-Pad6) -> /power/+BATTV
- Q2 pad 7: unconnected-(Q2-D_3-Pad7) -> /power/+BATTV
- Q2 pad 8: VMAIN -> /power/+BATTV
- Q2 pad 9: unconnected-(Q2-D_5-Pad9) -> /power/+BATTV
Routing:
- net /power/V_BASE: track 22.2 -> 0.92 mm, vias 12 -> 10
- net VMAIN: track 20.1 -> 1.61 mm, vias 19 -> 23
- net /power/+BATTV: track 11.9 -> 0.00 mm
- net /power/msft2: track 15.8 -> 6.03 mm, vias 10 -> 0
- net GND: track 21.1 -> 16.3 mm, vias 62 -> 58
- net /power/msft1: track 9.98 -> 7.09 mm, vias 8 -> 0
- net /power/VIN: track 1.46 -> 0.00 mm
- net /StepperA/MA2: vias 0 -> 10
- net /StepperA/MA1: vias 0 -> 7
- removed copper zone on B.Cu, net /power/msft1
- removed copper zone on F.Cu, net /power/msft1
- removed copper zone on B.Cu, net /power/msft2
- removed copper zone on F.Cu, net /power/msft2
