File: power.kicad_sch (KiCad schematic)
At the start: 27 parts, among them IC1 SiC437BED-T1-GE3, J4 XT60PW-M, Q1 PXP012-30QLJ, Q2 PXP012-30QLJ, U2 LTC4412xS6

Commit message: update
Parts:
- C21: footprint Capacitor_SMD:C_Elec_6.3x5.4 -> Capacitor_SMD:CP_Elec_10x10
- C6: footprint Capacitor_SMD:CP_Elec_10x12.5 -> Capacitor_SMD:C_Elec_8x10.2
Changed lines of the file:
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@@
 			)
 		)
-		(property "Footprint" "Capacitor_SMD:C_Elec_6.3x5.4"
+		(property "Footprint" "Capacitor_SMD:CP_Elec_10x10"
 			(at 240.03 86.36 0)
 			(effects
@@
 			)
 		)
-		(property "Footprint" "Capacitor_SMD:CP_Elec_10x12.5"
+		(property "Footprint" "Capacitor_SMD:C_Elec_8x10.2"
 			(at 110.49 67.31 0)
 			(effects
