File: power.kicad_sch (KiCad schematic)
At the start: 27 parts, among them IC1 SiC437BED-T1-GE3, J4 XT60PW-M, Q1 PXP012-30QLJ, Q2 PXP012-30QLJ, U2 LTC4412xS6

Commit message: update-i hate babs
Parts:
- L1: value 1.5uH -> 3.3uH; footprint Inductor_SMD:L_1008_2520Metric -> iclr:IND_SPM10065VT-3R3M-D
Connections:
- net GND: now also J4.2 (-)
- net V_BASE: now also C23.1
- removed net gnd_buff: C23.1, J4.2 (-)
Other:
- moved on the sheet: C23
Changed lines of the file:
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@@
 	)
 	(junction
+		(at 39.37 39.37)
+		(diameter 0)
+		(color 0 0 0 0)
+	)
+	(junction
 		(at 44.45 39.37)
 		(diameter 0)
@@
 	)
 	(junction
+		(at 36.83 50.8)
+		(diameter 0)
+		(color 0 0 0 0)
+	)
+	(junction
 		(at 171.45 90.17)
 		(diameter 0)
@@
 	(wire
 		(pts
+			(xy 36.83 41.91) (xy 36.83 50.8)
+		)
+		(stroke
+			(width 0)
+			(type default)
+		)
+	)
+	(wire
+		(pts
 			(xy 130.81 73.66) (xy 130.81 57.15)
 		)
@@
 	(wire
 		(pts
-			(xy 36.83 41.91) (xy 36.83 44.45)
-		)
-		(stroke
-			(width 0)
-			(type default)
-		)
-	)
-	(wire
-		(pts
 			(xy 148.59 58.42) (xy 148.59 62.23)
 		)
@@
 	(wire
 		(pts
-			(xy 36.83 39.37) (xy 44.45 39.37)
+			(xy 36.83 39.37) (xy 39.37 39.37)
 		)
 		(stroke
@@
 	(wire
 		(pts
-			(xy 36.83 50.8) (xy 36.83 49.53)
+			(xy 39.37 50.8) (xy 39.37 49.53)
 		)
 		(stroke
@@
 	(wire
 		(pts
+			(xy 39.37 44.45) (xy 39.37 39.37)
+		)
+		(stroke
+			(width 0)
+			(type default)
+		)
+	)
+	(wire
+		(pts
 			(xy 237.49 83.82) (xy 240.03 83.82)
 		)
@@
 	(wire
 		(pts
+			(xy 39.37 39.37) (xy 44.45 39.37)
+		)
+		(stroke
+			(width 0)
+			(type default)
+		)
+	)
+	(wire
+		(pts
 			(xy 194.31 34.29) (xy 194.31 38.1)
 		)
@@
 	(wire
 		(pts
+			(xy 39.37 50.8) (xy 36.83 50.8)
+		)
+		(stroke
+			(width 0)
+			(type default)
+		)
+	)
+	(wire
+		(pts
 			(xy 132.08 38.1) (xy 135.89 38.1)
 		)
@@
 		)
 	)
-	(label "gnd_buff"
-		(at 36.83 43.18 0)
-		(fields_autoplaced yes)
-		(effects
-			(font
-				(size 1.27 1.27)
-			)
-			(justify left bottom)
-		)
-	)
 	(label "msft1"
 		(at 57.15 43.18 0)
@@
 			)
 		)
-		(property "Value" "1.5uH"
+		(property "Value" "3.3uH"
 			(at 173.99 81.28 90)
 			(effects
@@
 			)
 		)
-		(property "Footprint" "Inductor_SMD:L_1008_2520Metric"
+		(property "Footprint" "iclr:IND_SPM10065VT-3R3M-D"
 			(at 173.99 83.82 0)
 			(effects
@@
 	(symbol
 		(lib_id "Device:C_Small")
-		(at 36.83 46.99 0)
+		(at 39.37 46.99 0)
 		(unit 1)
 		(exclude_from_sim no)
@@
 		(fields_autoplaced yes)
 		(property "Reference" "C23"
-			(at 39.37 45.7262 0)
+			(at 41.91 45.7262 0)
 			(effects
 				(font
@@
 		)
 		(property "Value" "0.1uF"
-			(at 39.37 48.2662 0)
+			(at 41.91 48.2662 0)
 			(effects
 				(font
@@
 		)
 		(property "Footprint" "Capacitor_SMD:C_0402_1005Metric"
-			(at 36.83 46.99 0)
+			(at 39.37 46.99 0)
 			(effects
 				(font
@@
 		)
 		(property "Datasheet" "~"
-			(at 36.83 46.99 0)
+			(at 39.37 46.99 0)
 			(effects
 				(font
@@
 		)
 		(property "Description" "Unpolarized capacitor, small symbol"
-			(at 36.83 46.99 0)
+			(at 39.37 46.99 0)
 			(effects
 				(font

Commit message: donedonedone
Parts:
- removed Q1, Q2: PXP012-30QLJ, iclr:PXP01230QLJ, symbol ICLR:PXP012-30QLJ
- added Q1, Q2: SQS141ELNW-T1_GE3, SQS850ENT1_GE3, symbol iclr:SQS141ELNW-T1_GE3
Connections:
- net VIN is gone; now on net VMAIN: IC1.22 (VIN_1), IC1.26 (VIN_2)
- net +BATTV: now also Q2.10, Q2.11, Q2.5, Q2.6, Q2.7, Q2.8, Q2.9
- net VMAIN: now also Q1.1, Q1.2, Q1.3, Q2.1, Q2.2, Q2.3
- net V_BASE: now also Q1.10, Q1.11, Q1.5, Q1.6, Q1.7, Q1.8, Q1.9
- net msft1: now also Q1.4
- net msft2: now also Q2.4
- no-connect marks 15 -> 12
