File: BetetrDom.kicad_sch (KiCad schematic)
At the start: 13 parts, among them J1 XT60PW-M, J2 Raspberry_Pi_2_3

Commit message: update
Changed lines of the file:
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@@
 	)
 	(label "Step1"
-		(at 44.45 101.6 0)
+		(at 44.45 101.6 180)
 		(fields_autoplaced yes)
 		(effects
@@
 				(size 1.27 1.27)
 			)
-			(justify left bottom)
+			(justify right bottom)
 		)
 	)

Commit message: update-i hate babs
Connections:
- net GND: now also J1.2 (-)
- net power/+BATTV: now also C5.1
- removed net gnd_buff: C5.1, J1.2 (-)
Other:
- moved on the sheet: C5
Changed lines of the file:
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@@
+	)
+	(junction
+		(at 36.83 59.69)
+		(diameter 0)
+		(color 0 0 0 0)
 	)
 	(junction
@@
 	)
 	(junction
+		(at 33.02 64.77)
+		(diameter 0)
+		(color 0 0 0 0)
+	)
+	(junction
 		(at 170.18 67.31)
 		(diameter 0)
@@
 	(wire
 		(pts
+			(xy 31.75 62.23) (xy 33.02 62.23)
+		)
+		(stroke
+			(width 0)
+			(type default)
+		)
+	)
+	(wire
+		(pts
 			(xy 34.29 109.22) (xy 34.29 107.95)
 		)
@@
 	(wire
 		(pts
-			(xy 31.75 63.5) (xy 31.75 62.23)
-		)
-		(stroke
-			(width 0)
-			(type default)
-		)
-	)
-	(wire
-		(pts
-			(xy 31.75 59.69) (xy 46.99 59.69)
+			(xy 31.75 59.69) (xy 36.83 59.69)
 		)
 		(stroke
@@
 	(wire
 		(pts
+			(xy 33.02 64.77) (xy 33.02 68.58)
+		)
+		(stroke
+			(width 0)
+			(type default)
+		)
+	)
+	(wire
+		(pts
+			(xy 33.02 68.58) (xy 31.75 68.58)
+		)
+		(stroke
+			(width 0)
+			(type default)
+		)
+	)
+	(wire
+		(pts
+			(xy 36.83 59.69) (xy 46.99 59.69)
+		)
+		(stroke
+			(width 0)
+			(type default)
+		)
+	)
+	(wire
+		(pts
+			(xy 36.83 64.77) (xy 33.02 64.77)
+		)
+		(stroke
+			(width 0)
+			(type default)
+		)
+	)
+	(wire
+		(pts
 			(xy 118.11 40.64) (xy 124.46 40.64)
+		)
+		(stroke
+			(width 0)
+			(type default)
+		)
+	)
+	(wire
+		(pts
+			(xy 33.02 62.23) (xy 33.02 64.77)
 		)
 		(stroke
@@
 			)
 			(justify right bottom)
-		)
-	)
-	(label "gnd_buff"
-		(at 31.75 62.23 0)
-		(fields_autoplaced yes)
-		(effects
-			(font
-				(size 1.27 1.27)
-			)
-			(justify left bottom)
 		)
 	)
@@
 	(symbol
 		(lib_id "Device:C_Small")
-		(at 31.75 66.04 0)
+		(at 36.83 62.23 0)
 		(unit 1)
 		(exclude_from_sim no)
@@
 		(fields_autoplaced yes)
 		(property "Reference" "C5"
-			(at 34.29 64.7762 0)
+			(at 39.37 60.9662 0)
 			(effects
 				(font
@@
 		)
 		(property "Value" "0.1uF"
-			(at 34.29 67.3162 0)
+			(at 39.37 63.5062 0)
 			(effects
 				(font
@@
 		)
 		(property "Footprint" "Capacitor_SMD:C_0402_1005Metric"
-			(at 31.75 66.04 0)
+			(at 36.83 62.23 0)
 			(effects
 				(font
@@
 		)
 		(property "Datasheet" "~"
-			(at 31.75 66.04 0)
+			(at 36.83 62.23 0)
 			(effects
 				(font
@@
 		)
 		(property "Description" "Unpolarized capacitor, small symbol"
-			(at 31.75 66.04 0)
-			(effects
-				(font
+			(at 36.83 62.23 0)
+			(effects
+				(font
